File: KeyboardPCB/KeyboardPCB.kicad_pcb (KiCad board)
At the start: 2 copper layers, 177 parts, among them SW0 RotaryEncoder_Switch

Commit message: Finished PCB v1
Parts:
- removed D88: ~, ScottoKeebs_Components:Diode_DO-35
- removed S16: ~, ScottoKeebs_MX:MX_PCB_1.00u
- SW0: footprint Connector_PinHeader_2.54mm:PinHeader_1x05_P2.54mm_Vertical -> ScottoKeebs_Scotto:Encoder_EC11_MX; moved to F.Cu
- moved SW0 228.9 mm to (363.5, 34.9), turned to 0 degrees
- moved A0 188.1 mm to (338.5, 101.6), turned to -90 degrees
- moved S75 35.9 mm to (285.0, 120.7)
- moved S76 35.9 mm to (344.5, 120.7)
- moved D12 35.9 mm to (292.1, 38.7)
- moved S15 35.9 mm to (344.5, 34.9)
- moved S30 35.9 mm to (292.1, 63.5)
- moved S32 35.9 mm to (344.5, 63.5)
- moved S33 35.9 mm to (363.5, 63.5)
- moved S47 35.9 mm to (296.9, 82.5)
- moved S49 35.9 mm to (344.5, 82.5)
- moved S50 35.9 mm to (363.5, 82.5)
- moved D62 35.9 mm to (268.3, 105.4)
- moved D83 35.9 mm to (285.0, 143.5)
- moved D84 35.9 mm to (308.8, 143.5)
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Connections:
- A0 pad 1: Row 0 -> Col 10
- A0 pad 10: Col 1 -> Col 8
- A0 pad 11: Col 2 -> Col 7
- A0 pad 12: Col 3 -> Col 15
- A0 pad 14: Col 4 -> Row 0
- A0 pad 15: Col 5 -> Row 1
- A0 pad 16: Col 6 -> DT
- A0 pad 17: Col 7 -> CLK
- A0 pad 19: Col 8 -> Col 16
- A0 pad 2: Row 1 -> Col 11
- A0 pad 20: Col 9 -> Row 2
- A0 pad 21: Col 10 -> Row 5
- A0 pad 22: Col 11 -> Row 4
- A0 pad 24: Col 12 -> Row 3
- A0 pad 25: Col 13 -> Col 0
- A0 pad 26: Col 14 -> Col 1
- A0 pad 27: Col 15 -> Col 2
- A0 pad 29: Col 16 -> Col 6
- A0 pad 30: unconnected-(A0-RUN-Pad30) -> NO
- A0 pad 31: CLK -> Col 5
- A0 pad 32: DT -> Col 4
- A0 pad 33: unconnected-(A0-AGND-Pad33) -> NO
- A0 pad 34: unconnected-(A0-GPIO28_ADC2-Pad34) -> Col 3
- A0 pad 35: unconnected-(A0-ADC_VREF-Pad35) -> NO
- A0 pad 36: unconnected-(A0-3V3-Pad36) -> NO
- A0 pad 37: unconnected-(A0-3V3_EN-Pad37) -> NO
- A0 pad 39: unconnected-(A0-VSYS-Pad39) -> NO
- A0 pad 4: Row 2 -> Col 12
- A0 pad 40: unconnected-(A0-VBUS-Pad40) -> NO
- A0 pad 5: Row 3 -> Col 13
- A0 pad 6: Row 4 -> Col 14
- A0 pad 7: Row 5 -> unconnected-(A0-GPIO5-Pad7)
- A0 pad 9: Col 0 -> Col 9
Routing:
- net Col 0: track 0.00 -> 434.1 mm
- net Row 0: track 0.00 -> 384.7 mm, vias 0 -> 1
- net Col 2: track 0.00 -> 380.6 mm
- net Col 1: track 0.00 -> 377.9 mm
- net Row 5: track 0.00 -> 362.0 mm
- net Row 1: track 0.00 -> 354.9 mm, vias 0 -> 1
- net Row 2: track 0.00 -> 329.7 mm
- net Col 3: track 0.00 -> 319.8 mm
- net Row 4: track 0.00 -> 313.3 mm
- net Row 3: track 0.00 -> 311.4 mm
- net Col 5: track 0.00 -> 308.8 mm
- net Col 4: track 0.00 -> 305.3 mm
- net Col 6: track 0.00 -> 278.8 mm
- net Col 8: track 0.00 -> 270.5 mm
- net Col 7: track 0.00 -> 266.9 mm
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- added copper zone on B.Cu, net (none)
- added copper zone on F.Cu, net (none)
Other:
- board outline added: 351 x 124.5 mm
- board text added: "//////// Winnand-TKL //////// Designed by: Aditya Itnal //////// github.com/winnand ////////"

Commit message: CAD Files
Routing:
- net GND: track 59.1 -> 0.00 mm, vias 1 -> 7
- net Col 16: track 108.6 -> 104.7 mm
- added copper zone on B.Cu, net GND
- added copper zone on F.Cu, net GND
- removed copper zone on B.Cu, net (none)
- removed copper zone on F.Cu, net (none)
Other:
- outline, holes or cut-outs redrawn

Commit message: added RGB header
Parts:
- added J1: Conn_01x04_Pin, Connector_PinHeader_2.54mm:PinHeader_1x04_P2.54mm_Vertical, B.Cu at (369.0, 116.4)
Connections:
- A0 pad 40: NO -> Net-(A0-VBUS)
- A0 pad 7: unconnected-(A0-GPIO5-Pad7) -> Net-(A0-GPIO5)
Routing:
- net Net-(A0-VBUS): track 0.00 -> 73.0 mm, vias 0 -> 3
- net Net-(A0-GPIO5): track 0.00 -> 61.6 mm
- net GND: track 0.00 -> 20.3 mm
Other:
- board size 351 x 124.5 mm -> 350.5 x 124.5 mm
- board text added: "G D +5v"
