File: KeyboardPCB/KeyboardPCB.kicad_sch (KiCad schematic)
At the start: 177 parts, among them SW0 RotaryEncoder_Switch

Commit message: Finished PCB v1
Parts:
- removed D88: ~, ScottoKeebs_Components:Diode_DO-35, symbol ScottoKeebs:Placeholder_Diode
- removed S16: ~, ScottoKeebs_MX:MX_PCB_1.00u, symbol ScottoKeebs:Placeholder_Keyswitch
- SW0: footprint Connector_PinHeader_2.54mm:PinHeader_1x05_P2.54mm_Vertical -> ScottoKeebs_Scotto:Encoder_EC11_MX
Connections:
- net CLK: now also A0.17 (GPIO13), SW0.B; no longer A0.31 (GPIO26_ADC0), SW0.A
- net Col 0: now also A0.25 (GPIO19); no longer A0.9 (GPIO6)
- net Col 1: now also A0.26 (GPIO20); no longer A0.10 (GPIO7)
- net Col 10: now also A0.1 (GPIO0); no longer A0.21 (GPIO16)
- net Col 11: now also A0.2 (GPIO1); no longer A0.22 (GPIO17)
- net Col 12: now also A0.4 (GPIO2); no longer A0.24 (GPIO18)
- net Col 13: now also A0.5 (GPIO3); no longer A0.25 (GPIO19)
- net Col 14: now also A0.6 (GPIO4); no longer A0.26 (GPIO20)
- net Col 15: now also A0.12 (GPIO9); no longer A0.27 (GPIO21)
- net Col 16: now also A0.19 (GPIO14), SW0.S1; no longer A0.29 (GPIO22), SW0.S2
- net Col 2: now also A0.27 (GPIO21); no longer A0.11 (GPIO8)
- net Col 3: now also A0.34 (GPIO28_ADC2); no longer A0.12 (GPIO9)
- net Col 4: now also A0.32 (GPIO27_ADC1); no longer A0.14 (GPIO10)
- net Col 5: now also A0.31 (GPIO26_ADC0); no longer A0.15 (GPIO11)
- net Col 6: now also A0.29 (GPIO22); no longer A0.16 (GPIO12)
- net Col 7: now also A0.11 (GPIO8); no longer A0.17 (GPIO13)
- net Col 8: now also A0.10 (GPIO7); no longer A0.19 (GPIO14)
- net Col 9: now also A0.9 (GPIO6); no longer A0.20 (GPIO15)
- net DT: now also A0.16 (GPIO12), SW0.A; no longer A0.32 (GPIO27_ADC1), SW0.B
- net Row 0: now also A0.14 (GPIO10); no longer A0.1 (GPIO0)
- net Row 1: now also A0.15 (GPIO11); no longer A0.2 (GPIO1)
- net Row 2: now also A0.20 (GPIO15); no longer A0.4 (GPIO2)
- net Row 3: now also A0.24 (GPIO18); no longer A0.5 (GPIO3)
- net Row 4: now also A0.22 (GPIO17); no longer A0.6 (GPIO4)
- net Row 5: now also A0.21 (GPIO16); no longer A0.7 (GPIO5)
- net at D16.2 (A): now also SW0.S2
- net NO: now reaches A0.30 (RUN)
- net NO: now also A0.33 (AGND), A0.35 (ADC_VREF), A0.36 (3V3), A0.37 (3V3_EN), A0.39 (VSYS), A0.40 (VBUS)
Other:
- moved on the sheet: SW0

Commit message: added RGB header
Parts:
- added J1: Conn_01x04_Pin, Connector_PinHeader_2.54mm:PinHeader_1x04_P2.54mm_Vertical, symbol Connector:Conn_01x04_Pin
Connections:
- net GND: now also J1.1 (Pin_1)
- net NO: no longer A0.40 (VBUS)
- net at A0.7 (GPIO5): now also J1.3 (Pin_3)
- new net: A0.40 (VBUS), J1.4 (Pin_4)
Changed lines of the file:
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@@
 	(wire
 		(pts
+			(xy 27.94 243.84) (xy 27.94 195.58)
+		)
+		(stroke
+			(width 0)
+			(type default)
+		)
+	)
+	(wire
+		(pts
 			(xy 157.48 83.82) (xy 170.18 83.82)
 		)
@@
 	(wire
 		(pts
+			(xy 62.23 151.13) (xy 118.11 151.13)
+		)
+		(stroke
+			(width 0)
+			(type default)
+		)
+	)
+	(wire
+		(pts
 			(xy 182.88 119.38) (xy 195.58 119.38)
 		)
@@
 	(wire
 		(pts
+			(xy 110.49 195.58) (xy 110.49 243.84)
+		)
+		(stroke
+			(width 0)
+			(type default)
+		)
+	)
+	(wire
+		(pts
 			(xy 132.08 83.82) (xy 144.78 83.82)
 		)
@@
 	(wire
 		(pts
+			(xy 110.49 243.84) (xy 27.94 243.84)
+		)
+		(stroke
+			(width 0)
+			(type default)
+		)
+	)
+	(wire
+		(pts
 			(xy 195.58 101.6) (xy 220.98 101.6)
 		)
@@
 	(wire
 		(pts
+			(xy 62.23 160.02) (xy 62.23 151.13)
+		)
+		(stroke
+			(width 0)
+			(type default)
+		)
+	)
+	(wire
+		(pts
 			(xy 215.9 38.1) (xy 215.9 55.88)
 		)
@@
 	(wire
 		(pts
+			(xy 27.94 195.58) (xy 39.37 195.58)
+		)
+		(stroke
+			(width 0)
+			(type default)
+		)
+	)
+	(wire
+		(pts
 			(xy 144.78 83.82) (xy 157.48 83.82)
 		)
@@
 	(wire
 		(pts
+			(xy 118.11 151.13) (xy 118.11 193.04)
+		)
+		(stroke
+			(width 0)
+			(type default)
+		)
+	)
+	(wire
+		(pts
 			(xy 81.28 66.04) (xy 93.98 66.04)
 		)
@@
 	(wire
 		(pts
+			(xy 118.11 193.04) (xy 130.81 193.04)
+		)
+		(stroke
+			(width 0)
+			(type default)
+		)
+	)
+	(wire
+		(pts
 			(xy 220.98 66.04) (xy 233.68 66.04)
 		)
@@
 	(wire
 		(pts
+			(xy 130.81 195.58) (xy 110.49 195.58)
+		)
+		(stroke
+			(width 0)
+			(type default)
+		)
+	)
+	(wire
+		(pts
 			(xy 228.6 55.88) (xy 228.6 73.66)
 		)
@@
 		)
 	)
+	(global_label "GND"
+		(shape input)
+		(at 130.81 200.66 180)
+		(fields_autoplaced yes)
+		(effects
+			(font
+				(size 1.27 1.27)
+			)
+			(justify right)
+		)
+		(property "Intersheetrefs" "${INTERSHEET_REFS}"
+			(at 123.9543 200.66 0)
+			(effects
+				(font
+					(size 1.27 1.27)
+				)
+				(justify right)
+				(hide yes)
+			)
+		)
+	)
 	(global_label "CLK"
 		(shape input)
@@
 		)
 	)
-	(global_label "NO"
-		(shape input)
-		(at 62.23 160.02 90)
-		(fields_autoplaced yes)
-		(effects
-			(font
-				(size 1.27 1.27)
-			)
-			(justify left)
-		)
-		(property "Intersheetrefs" "${INTERSHEET_REFS}"
-			(at 62.23 154.3738 90)
-			(effects
-				(font
-					(size 1.27 1.27)
-				)
-				(justify left)
-				(hide yes)
-			)
-		)
-	)
 	(global_label "Col 2"
 		(shape input)
@@
 					(unit 1)
 				)
+			)
+		)
+	)
+	(symbol
+		(lib_id "Connector:Conn_01x04_Pin")
+		(at 135.89 198.12 180)
+		(unit 1)
+		(exclude_from_sim no)
+		(in_bom yes)
+		(on_board yes)
+		(dnp no)
+		(fields_autoplaced yes)
+		(property "Reference" "J1"
+			(at 137.16 195.5799 0)
+			(effects
+				(font
+					(size 1.27 1.27)
+				)
+				(justify right)
+			)
+		)
+		(property "Value" "Conn_01x04_Pin"
+			(at 137.16 198.1199 0)
+			(effects
+				(font
+					(size 1.27 1.27)
+				)
+				(justify right)
+			)
+		)
+		(property "Footprint" "Connector_PinHeader_2.54mm:PinHeader_1x04_P2.54mm_Vertical"
+			(at 135.89 198.12 0)
+			(effects
+				(font
+					(size 1.27 1.27)
+				)
+				(hide yes)
+			)
+		)
+		(property "Datasheet" "~"
+			(at 135.89 198.12 0)
+			(effects
+				(font
+					(size 1.27 1.27)
+				)
+				(hide yes)
+			)
+		)
+		(property "Description" "Generic connector, single row, 01x04, script generated"
+			(at 135.89 198.12 0)
+			(effects
+				(font
+					(size 1.27 1.27)
+				)
+				(hide yes)
+			)
+		)
+		(pin "1"
+		)
+		(pin "4"
+		)
+		(pin "2"
+		)
+		(pin "3"
+		)
+		(instances
+			(project ""
+				(path "/27f9e1ed-2b10-4ded-8686-913ede2e8f33"
+					(reference "J1")
+					(unit 1)
+				)
